File: KiCAD/cl33mos.kicad_sch (KiCad schematic)
At the start: 13 parts, among them J1 USB_B_Micro, J2 Edge2x6_Connector, U2 ESP32-WROOM-32, U3 AMS1117-3.3

Commit message: Add svelte-based web interface (#31)
- Add svelte-based web UI developed with the help of claude.
- KiCAD update -> v1.3.  Change pump2 DIO, remove pump pull-downs
- board v1.3, test web page

The old interface can still be reached by at the "/root" path.
Connections:
- net P2: now also U2.16 (IO13); no longer U2.29 (IO5)
Changed lines of the file:
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@@
 (kicad_sch
-	(version 20231120)
+	(version 20250114)
 	(generator "eeschema")
-	(generator_version "8.0")
+	(generator_version "9.0")
 	(paper "A4")
 	(junction
@@
 	)
 	(no_connect
-		(at 110.49 83.82)
+		(at 110.49 78.74)
 	)
 	(no_connect
@@
 	(global_label "P2"
 		(shape input)
-		(at 110.49 78.74 0)
-		(fields_autoplaced yes)
-		(effects
-			(font
-				(size 1.27 1.27)
-			)
-			(justify left)
-		)
-		(property "Intersheetrefs" "${INTERSHEET_REFS}"
-			(at 115.9547 78.74 0)
-			(effects
-				(font
+		(at 110.49 83.82 0)
+		(fields_autoplaced yes)
+		(effects
+			(font
+				(size 1.27 1.27)
+			)
+			(justify left)
+		)
+		(property "Intersheetrefs" "${INTERSHEET_REFS}"
+			(at 115.9547 83.82 0)
+			(effects
+				(font
