File: KiCAD/Plant1337.kicad_pcb (KiCad board)
At the start: 4 copper layers, 59.1 x 41.9 mm, 63 parts, among them J1 USB_B_Micro, J2 Edge2x6_Connector, Q1 AO3400A, Q2 AO3400A, Q3 AO3400A, Q4 AO3400A, U1 SHTC3, U2 ESP32-WROOM-32, U3 AMS1117-3.3

Commit message: Add svelte-based web interface (#31)
- Add svelte-based web UI developed with the help of claude.
- KiCAD update -> v1.3.  Change pump2 DIO, remove pump pull-downs
- board v1.3, test web page

The old interface can still be reached by at the "/root" path.
Parts:
- removed REF** (x3): MountingHole_2.5mm, MountingHole:MountingHole_2.5mm
- removed Ru3, Ru4, Ru5, Ru6: 10k, Resistor_SMD:R_0603_1608Metric
Connections:
- U2 pad 16: unconnected-(U2-IO13-Pad16) -> P2
- U2 pad 29: P2 -> unconnected-(U2-IO5-Pad29)
Routing:
- net P2: track 42.6 -> 30.4 mm
- net GND: track 58.4 -> 50.4 mm
- net P3: track 47.1 -> 44.3 mm
- net Net-(Q4-G): track 3.99 -> 1.66 mm
- net Net-(Q2-G): track 3.72 -> 1.60 mm
- net Net-(Q1-G): track 3.81 -> 1.79 mm
- net Net-(Q3-G): track 4.20 -> 2.25 mm
Other:
- board text added: "Plantl337 v1.3 (c) Chris Lee"
- board text removed: "Plantl337 v1.2 (c) Chris Lee"

Commit message: Version update, board updates, stencil fixture (#32)
* KiCad updates, OpenSCAD design for PCB-stencil holder

* Added-back screw-holes at 2 corners of the board

* og3 -> 0.3.96
Parts:
- added REF**: MountingHole_2.5mm_stencil_hole, chl33_library:MountingHole_2.5mm_stencil_hole, F.Cu at (103.3, 62.5)
- added REF**: MountingHole_2.5mm_stencil_hole, chl33_library:MountingHole_2.5mm_stencil_hole, F.Cu at (49.8, 98.8)
Changed lines of the file:
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@@
 		)
 	)
+	(footprint "chl33_library:MountingHole_2.5mm_stencil_hole"
+		(locked yes)
+		(layer "F.Cu")
+		(at 103.251 62.484)
+		(descr "Mounting Hole 2.5mm, no annular")
+		(tags "mounting hole 2.5mm no annular")
+		(property "Reference" "REF**"
+			(at 0 -3.5 0)
+			(layer "F.SilkS")
+			(hide yes)
+			(effects
+				(font
+					(size 1 1)
+					(thickness 0.15)
+				)
+			)
+		)
+		(property "Value" "MountingHole_2.5mm_stencil_hole"
+			(at 0 3.5 0)
+			(layer "F.Fab")
+			(hide yes)
+			(effects
+				(font
+					(size 1 1)
+					(thickness 0.15)
+				)
+			)
+		)
+		(property "Datasheet" ""
+			(at 0 0 0)
+			(unlocked yes)
+			(layer "F.Fab")
+			(hide yes)
+			(effects
+				(font
+					(size 1.27 1.27)
+					(thickness 0.15)
+				)
+			)
+		)
+		(property "Description" ""
+			(at 0 0 0)
+			(unlocked yes)
+			(layer "F.Fab")
+			(hide yes)
+			(effects
+				(font
+					(size 1.27 1.27)
+					(thickness 0.15)
+				)
+			)
+		)
+		(attr exclude_from_pos_files exclude_from_bom)
+		(fp_circle
+			(center 0 0)
+			(end 2.5 0)
+			(stroke
+				(width 0.15)
+				(type solid)
+			)
+			(fill no)
+			(layer "Cmts.User")
+		)
+		(fp_circle
+			(center 0 0)
+			(end 2.75 0)
+			(stroke
+				(width 0.05)
+				(type solid)
+			)
+			(fill no)
+			(layer "F.CrtYd")
+		)
+		(fp_text user "${REFERENCE}"
+			(at 0 0 0)
+			(layer "F.Fab")
+			(effects
+				(font
+					(size 1 1)
+					(thickness 0.15)
+				)
+			)
+		)
+		(pad "" np_thru_hole circle
+			(at 0 0)
+			(size 2.5 2.5)
+			(drill 2.5)
+			(layers "F&B.Cu" "*.Paste" "*.Mask")
+		)
+		(embedded_fonts no)
+	)
 	(footprint "Diode_SMD:D_SMA"
 		(layer "F.Cu")
@@
 		)
 	)
+	(footprint "chl33_library:MountingHole_2.5mm_stencil_hole"
+		(locked yes)
+		(layer "F.Cu")
+		(at 49.784 98.806)
+		(descr "Mounting Hole 2.5mm, no annular")
+		(tags "mounting hole 2.5mm no annular")
+		(property "Reference" "REF**"
+			(at 0 -3.5 0)
+			(layer "F.SilkS")
+			(hide yes)
+			(effects
+				(font
+					(size 1 1)
+					(thickness 0.15)
+				)
+			)
+		)
+		(property "Value" "MountingHole_2.5mm_stencil_hole"
+			(at 0 3.5 0)
+			(layer "F.Fab")
+			(hide yes)
+			(effects
+				(font
+					(size 1 1)
+					(thickness 0.15)
+				)
+			)
+		)
+		(property "Datasheet" ""
+			(at 0 0 0)
+			(unlocked yes)
+			(layer "F.Fab")
+			(hide yes)
+			(effects
+				(font
+					(size 1.27 1.27)
+					(thickness 0.15)
+				)
+			)
+		)
+		(property "Description" ""
+			(at 0 0 0)
+			(unlocked yes)
+			(layer "F.Fab")
+			(hide yes)
+			(effects
+				(font
+					(size 1.27 1.27)
+					(thickness 0.15)
+				)
+			)
+		)
+		(attr exclude_from_pos_files exclude_from_bom)
+		(fp_circle
+			(center 0 0)
+			(end 2.5 0)
+			(stroke
+				(width 0.15)
+				(type solid)
+			)
+			(fill no)
+			(layer "Cmts.User")
+		)
+		(fp_circle
+			(center 0 0)
+			(end 2.75 0)
+			(stroke
+				(width 0.05)
+				(type solid)
+			)
+			(fill no)
+			(layer "F.CrtYd")
+		)
+		(fp_text user "${REFERENCE}"
+			(at 0 0 0)
+			(layer "F.Fab")
+			(effects
+				(font
+					(size 1 1)
+					(thickness 0.15)
+				)
+			)
+		)
+		(pad "" np_thru_hole circle
+			(at 0 0)
+			(size 2.5 2.5)
+			(drill 2.5)
+			(layers "F&B.Cu" "*.Paste" "*.Mask")
+		)
+		(embedded_fonts no)
+	)
 	(footprint "Resistor_SMD:R_0603_1608Metric"
